Commit message: atlas walking with pinocchio lib (change was zeroing joint frictions and link dampings)

File: robot_model/atlas/atlas_v4_with_multisense.urdf (robot description, URDF)
Before this commit: robot multisense_sl, 33 links, 32 joints
Links:
- added link pelvis_com, mass 0.001
Joints:
- added joint pelvis_com_fixed: type fixed, parent pelvis, child pelvis_com, origin xyz=0.0111 0 0.0271 rpy=0 -0 0

File: robot_model/atlas/atlas_v4_with_multisense_relative_path.urdf (robot description, URDF)
Before this commit: robot multisense_sl, 33 links, 32 joints
Links:
- added link pelvis_com, mass 0.001
Joints:
- added joint pelvis_com_fixed: type fixed, parent pelvis, child pelvis_com, origin xyz=0.0111 0 0.0271 rpy=0 -0 0
