Commit message: valkyrie model modified, valkyrie crbi_trainer added

File: robot_model/valkyrie/valkyrie.urdf (robot description, URDF)
Before this commit: robot valkyrie, 46 links, 45 joints
Links:
- link head: geometry 
- link hokuyo_link: geometry visual mesh filename=package://meshes/multisense/head_camera.obj
- link leftAnklePitchLink: geometry visual mesh filename=package://meshes/legs/lj5.obj
- link leftElbowPitchLink: geometry visual mesh filename=package://meshes/arms/left_elbow_mass_sim.obj
- link leftFoot: geometry collision box size=0.27 0.16 0.064; visual mesh filename=package://meshes/legs/foot_texture.obj
- link leftHipPitchLink: geometry visual mesh filename=package://meshes/legs/lj3_left_texture.obj
- link leftHipRollLink: geometry visual mesh filename=package://meshes/legs/lj2_left_texture.obj
- link leftHipYawLink: geometry visual mesh filename=package://meshes/legs/lj1_left.obj
- link leftKneePitchLink: geometry visual mesh filename=package://meshes/legs/lj4_left_texture.obj
- link leftShoulderPitchLink: geometry visual mesh filename=package://meshes/arms/aj1_left.obj
- link leftShoulderRollLink: geometry visual mesh filename=package://meshes/arms/aj2_left_texture.obj
- link leftShoulderYawLink: geometry visual mesh filename=package://meshes/arms/aj3_left_texture.obj
- link lowerNeckPitchLink: geometry visual mesh filename=package://meshes/head/neckj1.obj
- link neckYawLink: geometry visual mesh filename=package://meshes/head/neckj2.obj
- link pelvis: geometry visual mesh filename=package://meshes/pelvis/pelvis.obj
- link rightAnklePitchLink: geometry visual mesh filename=package://meshes/legs/lj5_texture.obj
- link rightElbowPitchLink: geometry visual mesh filename=package://meshes/arms/right_elbow_mass_sim.obj
- link rightFoot: geometry collision box size=0.27 0.16 0.064; visual mesh filename=package://meshes/legs/foot_texture.obj
- link rightHipPitchLink: geometry visual mesh filename=package://meshes/legs/lj3_right_texture.obj
- link rightHipRollLink: geometry visual mesh filename=package://meshes/legs/lj2_right_texture.obj
- link rightHipYawLink: geometry visual mesh filename=package://meshes/legs/lj1_right.obj
- link rightKneePitchLink: geometry visual mesh filename=package://meshes/legs/lj4_right_texture.obj
- link rightShoulderPitchLink: geometry visual mesh filename=package://meshes/arms/aj1_right.obj
- link rightShoulderRollLink: geometry visual mesh filename=package://meshes/arms/aj2_right_texture.obj
- link rightShoulderYawLink: geometry visual mesh filename=package://meshes/arms/aj3_right_texture.obj
- link torso: geometry visual mesh filename=package://meshes/torso/torso_textured.obj
- link torsoPitchLink: geometry visual mesh filename=package://meshes/torso/torsopitch.obj
- link torsoYawLink: geometry visual mesh filename=package://meshes/torso/torsoyaw.obj
- link upperNeckPitchLink: geometry visual mesh filename=package://meshes/head/head_multisense_visor_textured.obj
