Commit message: slope added

File: robot_model/ground/slope.urdf (robot description, URDF)
Before this commit: robot stair, 2 links, 1 joints
Links:
- link baseLink: geometry visual box size=0.304 0.6 0.304
- link secondLink: geometry visual box size=0.304 0.6 0.304
Joints:
- joint j0: axis 0 0 1 -> (none); origin xyz=0.35 0 0. rpy=0 0 0 -> xyz=0.25 0 0 rpy=0 0 0
