Commit message: atlas chimney jump added

File: robot_model/ground/chimney.urdf (robot description, URDF)
Before this commit: robot chimney, 4 links, 3 joints
Links:
- removed link third_ground
Joints:
- removed joint first_to_third
- joint first_to_fourth: origin xyz=1.1 0 0 rpy=0 0 0 -> xyz=0.7 0 0 rpy=0 0 0
- joint first_to_second: origin xyz=0.329 0 0.08 rpy=0 0 0 -> xyz=0.352 0 0.08 rpy=0 0 0
