Commit message: debugging draco3 pnc

File: robot_model/manipulator/rolling_joint.urdf (robot description, URDF)
Before this commit: robot rolling_joint, 5 links, 4 joints
Joints:
- joint j0: limit (none) -> lower=-6.28318530718 upper=6.28318530718 effort=150.0 velocity=3.15; origin (none) -> xyz=1 0 0 rpy=0 0 0; type fixed -> revolute
