Commit message: working on laikago

File: robot_model/laikago/laikago_toes.urdf (robot description, URDF)
Before this commit: robot plane, 17 links, 16 joints
Links:
- link FL_hip_motor: geometry visual mesh filename=hip_motor.obj scale=1 1 1
- link FL_lower_leg: geometry visual mesh filename=lower_leg3.obj scale=1 1 1
- link FL_upper_leg: geometry visual mesh filename=upper_leg_left.obj scale=1 1 1
- link FR_hip_motor: geometry visual mesh filename=hip_motor_mirror.obj scale=1 1 1
- link FR_lower_leg: geometry visual mesh filename=lower_leg3.obj scale=1 1 1
- link FR_upper_leg: geometry visual mesh filename=upper_leg_mirror.obj scale=1 1 1
- link chassis: geometry visual mesh filename=chassis.obj scale=1 1 1

Commit message: laikago pnc draft, debugging

File: robot_model/laikago/laikago_toes.urdf (robot description, URDF)
Before this commit: robot plane, 17 links, 16 joints
Links:
- link FL_hip_motor: geometry visual mesh filename=package://hip_motor.obj scale=1 1 1
- link FL_lower_leg: geometry visual mesh filename=package://lower_leg3.obj scale=1 1 1
- link FL_upper_leg: geometry visual mesh filename=package://upper_leg_left.obj scale=1 1 1
- link FR_hip_motor: geometry visual mesh filename=package://hip_motor_mirror.obj scale=1 1 1
- link FR_lower_leg: geometry visual mesh filename=package://lower_leg3.obj scale=1 1 1
- link FR_upper_leg: geometry visual mesh filename=package://upper_leg_mirror.obj scale=1 1 1
- link RL_hip_motor: geometry visual mesh filename=package://hip_motor.obj scale=1 1 1
- link RL_lower_leg: geometry visual mesh filename=package://lower_leg3.obj scale=1 1 1
- link RL_upper_leg: geometry visual mesh filename=package://upper_leg_left2.obj scale=1 1 1
- link RR_hip_motor: geometry visual mesh filename=package://hip_motor_mirror.obj scale=1 1 1
- link RR_lower_leg: geometry visual mesh filename=package://lower_leg3.obj scale=1 1 1
- link RR_upper_leg: geometry visual mesh filename=package://upper_leg_mirror2.obj scale=1 1 1
- link chassis: geometry visual mesh filename=package://chassis.obj scale=1 1 1
Joints:
- joint FL_hip_motor_2_chassis_joint: type continuous -> revolute
- joint FL_lower_leg_2_upper_leg_joint: type continuous -> revolute
- joint FL_upper_leg_2_hip_motor_joint: type continuous -> revolute
- joint FR_hip_motor_2_chassis_joint: type continuous -> revolute
- joint FR_lower_leg_2_upper_leg_joint: type continuous -> revolute
- joint FR_upper_leg_2_hip_motor_joint: type continuous -> revolute
- joint RL_hip_motor_2_chassis_joint: type continuous -> revolute
- joint RL_lower_leg_2_upper_leg_joint: type continuous -> revolute
- joint RL_upper_leg_2_hip_motor_joint: type continuous -> revolute
- joint RR_hip_motor_2_chassis_joint: type continuous -> revolute
- joint RR_lower_leg_2_upper_leg_joint: type continuous -> revolute
- joint RR_upper_leg_2_hip_motor_joint: type continuous -> revolute
