Commit message: bookshelf urdf for draco

File: robot_model/bookcase/blue_can.urdf (robot description, URDF)
Before this commit: robot blue_can, 1 links, 0 joints
Links:
- link can: geometry collision cylinder length=0.1 radius=0.05; visual cylinder length=0.1 radius=0.05

File: robot_model/bookcase/bookshelf.urdf (robot description, URDF)
Before this commit: robot bookcase, 9 links, 8 joints
Links:
- link back: geometry visual box size=2.1 0.02 1.5
- link base: geometry collision box size=2.0 0.3 0.05; visual box size=2.0 0.3 0.05
- link leftSide: geometry visual box size=0.05 0.3 1.5
- link rightSide: geometry visual box size=0.05 0.3 1.5
- link shelf1: geometry collision box size=2.0 0.3 0.05; visual box size=2.0 0.3 0.05
- link shelf2: geometry collision box size=2.0 0.3 0.05; visual box size=2.0 0.3 0.05
- link shelf3: geometry collision box size=2.0 0.3 0.05; visual box size=2.0 0.3 0.05
- link shelf4: geometry collision box size=2.0 0.3 0.05; visual box size=2.0 0.3 0.05
- link top: geometry collision box size=2.0 0.3 0.05; visual box size=2.0 0.3 0.05
Joints:
- joint j0: origin xyz=0.5 0 -0.025 rpy=0 0 0 -> xyz=1 0 -0.025 rpy=0 0 0
- joint j1: origin xyz=-0.5 0 -0.025 rpy=0 0 0 -> xyz=-1 0 -0.025 rpy=0 0 0
- joint j2: origin xyz=-0.5 0 0.4 rpy=0 0 0 -> xyz=-1 0 0.3 rpy=0 0 0
- joint j3: origin xyz=-0.5 0 0.8 rpy=0 0 0 -> xyz=-1 0 0.6 rpy=0 0 0
- joint j4: origin xyz=-0.5 0 1.2 rpy=0 0 0 -> xyz=-1 0 0.9 rpy=0 0 0
- joint j5: origin xyz=-0.5 0 1.6 rpy=0 0 0 -> xyz=-1 0 1.2 rpy=0 0 0
- joint j6: origin xyz=-0.5 0 2 rpy=0 0 0 -> xyz=-1 0 1.5 rpy=0 0 0

File: robot_model/bookcase/green_can.urdf (robot description, URDF)
Before this commit: robot green_can, 1 links, 0 joints
Links:
- link can: geometry collision cylinder length=0.15 radius=0.05; visual cylinder length=0.15 radius=0.05

File: robot_model/bookcase/red_can.urdf (robot description, URDF)
Before this commit: robot red_can, 1 links, 0 joints
Links:
- link can: geometry collision cylinder length=0.15 radius=0.075; visual cylinder length=0.15 radius=0.075

Commit message: grabbing can

File: robot_model/bookcase/blue_can.urdf (robot description, URDF)
Before this commit: robot blue_can, 1 links, 0 joints
Links:
- link can: mass 0.1 -> 0.75; geometry collision box size=0.1 0.1 0.15; visual box size=0.12 0.12 0.15
