Commit message: Have correct transform sent to vision, swapped back to rgb+depth topics - much faster

File: robot_model/bookcase/bookshelf.urdf (robot description, URDF)
Before this commit: robot bookcase, 9 links, 8 joints
Links:
- link base: geometry collision box size=2.0 1.0 0.05; visual box size=2.0 1.0 0.05
- link leftSide: geometry visual box size=0.05 1.0 1.5
- link rightSide: geometry visual box size=0.05 1.0 1.5
- link shelf1: geometry collision box size=2.0 1.0 0.05; visual box size=2.0 1.0 0.05
- link shelf2: geometry collision box size=2.0 1.0 0.05; visual box size=2.0 1.0 0.05
- link shelf3: geometry collision box size=2.0 1.0 0.05; visual box size=2.0 1.0 0.05
- link shelf4: geometry collision box size=2.0 1.0 0.05; visual box size=2.0 1.0 0.05
- link top: geometry collision box size=2.0 1.0 0.05; visual box size=2.0 1.0 0.05
