Commit message: scene changes, stub for safety assessment function

File: robot_model/bookcase/prop3.urdf (robot description, URDF)
Before this commit: robot blue_can, 1 links, 0 joints
Links:
- link can: mass 0.01 -> 0.1; geometry collision cylinder length=0.15 radius=0.05; visual cylinder length=0.15 radius=0.05

File: robot_model/bookcase/prop6.urdf (robot description, URDF)
Before this commit: robot blue_can, 1 links, 0 joints
Links:
- link can: mass 0.01 -> 0.1; geometry collision cylinder length=0.15 radius=0.05; visual cylinder length=0.15 radius=0.05
