Commit message: Added safety assessment function to rosnode, scene changes premerge

File: robot_model/bookcase/prop4.urdf (robot description, URDF)
Before this commit: robot blue_can, 1 links, 0 joints
Links:
- link can: geometry collision cylinder length=0.15 radius=0.075; visual cylinder length=0.15 radius=0.075

File: robot_model/bookcase/red_can.urdf (robot description, URDF)
Before this commit: robot red_can, 1 links, 0 joints
Links:
- link can: geometry collision box size=0.1 0.1 0.15; visual box size=0.12 0.12 0.15
