Commit message: gripper test done

File: robot_model/ezgripper/gripper.urdf (robot description, URDF)
Before this commit: robot gripper, 5 links, 4 joints
Links:
- added link basePosX, mass 0.00000001
- added link basePosY, mass 0.00000001
- added link world; visual box size=0.001 0.001 0.001
Joints:
- added joint basePosX: type prismatic, parent world, child basePosX, origin xyz=0 0 0 rpy=0 0 0, axis 1 0 0, limit lower=-200. upper=200. effort=150.0 velocity=100.0
- added joint basePosY: type prismatic, parent basePosX, child basePosY, origin xyz=0 0 0 rpy=0 0 0, axis 0 1 0, limit lower=-200. upper=200. effort=150.0 velocity=100.0
- added joint basePosZ: type prismatic, parent basePosY, child left_ezgripper_palm_link, origin xyz=0 0 0 rpy=0 0 0, axis 0 0 1, limit lower=-200. upper=200. effort=150.0 velocity=100.0
