Commit message: rewrite state machines

File: robot_model/draco3/draco3_gripper.urdf (robot description, URDF)
Before this commit: robot draco_3, 45 links, 44 joints
Links:
- added link l_hand_contact, mass 1e-9; visual sphere radius=0.01
- added link r_hand_contact, mass 1e-9; visual sphere radius=0.01
Joints:
- added joint l_hand_contact_frame: type fixed, parent l_sake_gripper_link, child l_hand_contact, origin xyz=0 0 -0.150052 rpy=0 0 0, axis 0 0 0
- added joint r_hand_contact_frame: type fixed, parent r_sake_gripper_link, child r_hand_contact, origin xyz=0 0 -0.150052 rpy=0 0 0, axis 0 0 0
