Commit message: add draco3_pnc, but not verified yet

File: robot_model/draco3/draco3.urdf (robot description, URDF)
Before this commit: robot draco_3, 36 links, 35 joints
Links:
- added link torso_com_link, mass 1e-9
Joints:
- added joint torso_com: type fixed, parent torso_link, child torso_com_link, origin xyz=-0.0310745 -0.000497416 0.137484 rpy=0 0 0

Commit message: validating camera location, segfault when adding camera link (need to be debug)

File: robot_model/draco3/draco3.urdf (robot description, URDF)
Before this commit: robot draco_3, 37 links, 36 joints
Links:
- added link l_camera, mass 1e-9; visual sphere radius=0.01
- added link r_camera, mass 1e-9; visual sphere radius=0.01
Joints:
- added joint l_camera_frame: type fixed, parent l_sake_gripper_link, child l_camera, origin xyz=-0.05535 0 -0.073 rpy=0 3.14 0, axis 0 0 0
- added joint r_camera_frame: type fixed, parent r_sake_gripper_link, child r_camera, origin xyz=-0.05535 0 -0.073 rpy=0 3.14 0, axis 0 0 0
- joint r_hand_contact_frame: origin xyz=0 0 -0.150052 rpy=-1.2326e-31 1.26435e-32 -2.84264e-31 -> xyz=0 0 -0.150052 rpy=0 0 0

Commit message: foot enlarged, finding parameters for walking

File: robot_model/draco3/draco3.urdf (robot description, URDF)
Before this commit: robot draco_3, 39 links, 38 joints
Links:
- link l_ankle_ie_link: geometry collision box size=0.25 0.15 0.0591; visual mesh filename=package://meshes/l_ankle_ie_link.stl
- link r_ankle_ie_link: geometry collision box size=0.25 0.15 0.0591; visual mesh filename=package://meshes/r_ankle_ie_link.stl

File: robot_model/draco3/draco3_gripper.urdf (robot description, URDF)
Before this commit: robot draco_3, 45 links, 44 joints
Links:
- link l_ankle_ie_link: geometry collision box size=0.25 0.15 0.0591; visual mesh filename=package://meshes/l_ankle_ie_link.stl
- link r_ankle_ie_link: geometry collision box size=0.25 0.15 0.0591; visual mesh filename=package://meshes/r_ankle_ie_link.stl

Commit message: add camera frame / hand contact frame. before visualizing target frame

File: robot_model/draco3/draco3.urdf (robot description, URDF)
Before this commit: robot draco_3, 39 links, 38 joints
Joints:
- joint l_hand_contact_frame: origin xyz=0 0 -0.150052 rpy=0 0 0 -> xyz=0 0 -0.2 rpy=0 0 0
- joint r_hand_contact_frame: origin xyz=0 0 -0.150052 rpy=0 0 0 -> xyz=0 0 -0.2 rpy=0 0 0

File: robot_model/draco3/draco3_gripper.urdf (robot description, URDF)
Before this commit: robot draco_3, 47 links, 46 joints
Links:
- added link camera, mass 1e-9; visual sphere radius=0.001
- link l_hand_contact: geometry visual sphere radius=0.001
- link r_hand_contact: geometry visual sphere radius=0.001
Joints:
- added joint camera_frame: type fixed, parent neck_pitch_link, child camera, origin xyz=0.08 0 0.08 rpy=0 0 0, axis 0 0 0
- joint l_hand_contact_frame: origin xyz=0 0 -0.150052 rpy=0 0 0 -> xyz=0 0 -0.2 rpy=0 0 0
- joint r_hand_contact_frame: origin xyz=0 0 -0.150052 rpy=0 0 0 -> xyz=0 0 -0.2 rpy=0 0 0

Commit message: draco3 double support hand returning state machine added

File: robot_model/draco3/draco3.urdf (robot description, URDF)
Before this commit: robot draco_3, 39 links, 38 joints
Links:
- link l_hip_fe_link: geometry visual mesh filename=package://meshes/l_hip_fe_link3.obj
- link l_knee_fe_ld: geometry visual mesh filename=package://meshes/l_knee_fe_ld3.obj
- link l_shoulder_ie_link: geometry visual mesh filename=package://meshes/l_shoulder_ie_link3.obj
- link neck_pitch_link: geometry visual mesh filename=package://meshes/neck_pitch_link3.obj
- link r_hip_fe_link: geometry visual mesh filename=package://meshes/r_hip_fe_link3.obj
- link r_knee_fe_ld: geometry visual mesh filename=package://meshes/r_knee_fe_ld3.obj
- link r_shoulder_ie_link: geometry visual mesh filename=package://meshes/r_shoulder_ie_link3.obj
- link torso_link: geometry visual mesh filename=package://meshes/torso_link3.obj

Commit message: renamed draco3.urdf (exploded robot view) -> draco3_pin_mdel.urdf and draco3_gripper_mesh_updated.urdf -> draco3.urdf

File: robot_model/draco3/draco3.urdf (robot description, URDF)
Before this commit: robot draco_3, 39 links, 38 joints
Links:
- removed link l_camera
- removed link r_camera
- added link camera, mass 1e-9; visual sphere radius=0.001
- added link left_ezgripper_finger_L1_1, mass .025; visual mesh filename=package://meshes/ezgripper_gen2/SAKE_Finger_L1_Gen2.stl
- added link left_ezgripper_finger_L1_2, mass .025; visual mesh filename=package://meshes/ezgripper_gen2/SAKE_Finger_L1_Gen2.stl
- added link left_ezgripper_finger_L2_1, mass .025; collision mesh filename=package://meshes/ezgripper_gen2/SAKE_Finger_L2_Gen2.stl; visual mesh filename=package://meshes/ezgripper_gen2/SAKE_Finger_L2_Gen2.stl
- added link left_ezgripper_finger_L2_2, mass .025; collision mesh filename=package://meshes/ezgripper_gen2/SAKE_Finger_L2_Gen2.stl; visual mesh filename=package://meshes/ezgripper_gen2/SAKE_Finger_L2_Gen2.stl
- added link left_ezgripper_palm_link, mass .3; visual mesh filename=package://meshes/ezgripper_gen2/SAKE_Palm_Dual_Gen2.stl
- added link right_ezgripper_finger_L1_1, mass .025; visual mesh filename=package://meshes/ezgripper_gen2/SAKE_Finger_L1_Gen2.stl
- added link right_ezgripper_finger_L1_2, mass .025; visual mesh filename=package://meshes/ezgripper_gen2/SAKE_Finger_L1_Gen2.stl
- added link right_ezgripper_finger_L2_1, mass .025; collision mesh filename=package://meshes/ezgripper_gen2/SAKE_Finger_L2_Gen2.stl; visual mesh filename=package://meshes/ezgripper_gen2/SAKE_Finger_L2_Gen2.stl
- added link right_ezgripper_finger_L2_2, mass .025; collision mesh filename=package://meshes/ezgripper_gen2/SAKE_Finger_L2_Gen2.stl; visual mesh filename=package://meshes/ezgripper_gen2/SAKE_Finger_L2_Gen2.stl
- added link right_ezgripper_palm_link, mass .3; visual mesh filename=package://meshes/ezgripper_gen2/SAKE_Palm_Dual_Gen2.stl
- link l_hand_contact: geometry visual sphere radius=0.001
- link l_sake_gripper_link: mass 0.545 -> 0.145; geometry visual mesh filename=package://meshes/l_sake_gripper_mount.stl
- link r_hand_contact: geometry visual sphere radius=0.001
- link r_sake_gripper_link: mass 0.545 -> 0.145; geometry visual mesh filename=package://meshes/r_sake_gripper_mount.stl
Joints:
- removed joint l_camera_frame
- removed joint r_camera_frame
- added joint camera_frame: type fixed, parent neck_pitch_link, child camera, origin xyz=0.08 0 0.08 rpy=0 0 0, axis 0 0 0
- added joint l_wrist_mount2: type fixed, parent l_wrist_pitch_link, child left_ezgripper_palm_link, origin xyz=0 0 -0.053 rpy=0 1.57 0
- added joint left_ezgripper_knuckle_L1_L2_1: type revolute, parent left_ezgripper_finger_L1_1, child left_ezgripper_finger_L2_1, origin xyz=0.052 0 0 rpy=0 0 0, axis 0 1 0, limit lower=0 upper=1.94 effort=1 velocity=3.67
- added joint left_ezgripper_knuckle_L1_L2_2: type revolute, parent left_ezgripper_finger_L1_2, child left_ezgripper_finger_L2_2, origin xyz=0.052 0 0 rpy=0 0 0, axis 0 1 0, limit lower=0 upper=1.94 effort=1 velocity=3.67
- added joint left_ezgripper_knuckle_palm_L1_1: type revolute, parent left_ezgripper_palm_link, child left_ezgripper_finger_L1_1, origin xyz=0.072569 0.03 0 rpy=-1.5708 0 1.57075, axis 0 1 0, limit lower=0 upper=1.94 effort=1 velocity=3.67
- added joint left_ezgripper_knuckle_palm_L1_2: type revolute, parent left_ezgripper_palm_link, child left_ezgripper_finger_L1_2, origin xyz=0.072569 -0.03 0 rpy=1.5708 0 -1.57075, axis 0 1 0, limit lower=0 upper=1.94 effort=1 velocity=3.67
- added joint r_wrist_mount2: type fixed, parent r_wrist_pitch_link, child right_ezgripper_palm_link, origin xyz=0 0 -0.053 rpy=0 1.57 0
- added joint right_ezgripper_knuckle_L1_L2_1: type revolute, parent right_ezgripper_finger_L1_1, child right_ezgripper_finger_L2_1, origin xyz=0.052 0 0 rpy=0 0 0, axis 0 1 0, limit lower=0 upper=1.94 effort=1 velocity=3.67
- added joint right_ezgripper_knuckle_L1_L2_2: type revolute, parent right_ezgripper_finger_L1_2, child right_ezgripper_finger_L2_2, origin xyz=0.052 0 0 rpy=0 0 0, axis 0 1 0, limit lower=0 upper=1.94 effort=1 velocity=3.67
- added joint right_ezgripper_knuckle_palm_L1_1: type revolute, parent right_ezgripper_palm_link, child right_ezgripper_finger_L1_1, origin xyz=0.072569 0.03 0 rpy=-1.5708 0 1.57075, axis 0 1 0, limit lower=0 upper=1.94 effort=1 velocity=3.67
- added joint right_ezgripper_knuckle_palm_L1_2: type revolute, parent right_ezgripper_palm_link, child right_ezgripper_finger_L1_2, origin xyz=0.072569 -0.03 0 rpy=1.5708 0 -1.57075, axis 0 1 0, limit lower=0 upper=1.94 effort=1 velocity=3.67

File: robot_model/draco3/draco3_pin_model.urdf (robot description, URDF)
Before this commit: robot draco_3, 48 links, 47 joints
Links:
- removed link camera
- removed link left_ezgripper_finger_L1_1
- removed link left_ezgripper_finger_L1_2
- removed link left_ezgripper_finger_L2_1
- removed link left_ezgripper_finger_L2_2
- removed link left_ezgripper_palm_link
- removed link right_ezgripper_finger_L1_1
- removed link right_ezgripper_finger_L1_2
- removed link right_ezgripper_finger_L2_1
- removed link right_ezgripper_finger_L2_2
- removed link right_ezgripper_palm_link
- added link l_camera, mass 1e-9; visual sphere radius=0.01
- added link r_camera, mass 1e-9; visual sphere radius=0.01
- link l_hand_contact: geometry 
- link l_sake_gripper_link: mass 0.145 -> 0.545; geometry visual mesh filename=package://meshes/l_sake_gripper_link.stl
- link r_hand_contact: geometry 
- link r_sake_gripper_link: mass 0.145 -> 0.545; geometry visual mesh filename=package://meshes/r_sake_gripper_link.stl
Joints:
- removed joint camera_frame
- removed joint l_wrist_mount2
- removed joint left_ezgripper_knuckle_L1_L2_1
- removed joint left_ezgripper_knuckle_L1_L2_2
- removed joint left_ezgripper_knuckle_palm_L1_1
- removed joint left_ezgripper_knuckle_palm_L1_2
- removed joint r_wrist_mount2
- removed joint right_ezgripper_knuckle_L1_L2_1
- removed joint right_ezgripper_knuckle_L1_L2_2
- removed joint right_ezgripper_knuckle_palm_L1_1
- removed joint right_ezgripper_knuckle_palm_L1_2
- added joint l_camera_frame: type fixed, parent l_sake_gripper_link, child l_camera, origin xyz=-0.05535 0 -0.073 rpy=0 3.14 0, axis 0 0 0
- added joint r_camera_frame: type fixed, parent r_sake_gripper_link, child r_camera, origin xyz=-0.05535 0 -0.073 rpy=0 3.14 0, axis 0 0 0
